File: mysplitKeeb/mysplitKeeb.kicad_pcb (KiCad board)
At the start: 2 copper layers, 35 parts, among them Q1 Q_PNP_EBC, Q10 Q_PNP_EBC, Q11 Q_PNP_EBC, Q12 Q_PNP_EBC, Q13 Q_PNP_EBC, Q14 Q_PNP_EBC, Q15 Q_PNP_EBC, Q16 Q_PNP_EBC, Q17 Q_PNP_EBC, Q18 Q_PNP_EBC, Q19 Q_PNP_EBC, Q2 Q_PNP_EBC, Q20 Q_PNP_EBC, Q21 Q_PNP_EBC, Q22 Q_PNP_EBC, Q23 Q_PNP_EBC, Q24 Q_PNP_EBC, Q25 Q_PNP_EBC, Q26 Q_PNP_EBC, Q27 Q_PNP_EBC, Q28 Q_PNP_EBC, Q29 Q_PNP_EBC, Q3 Q_PNP_EBC, Q30 Q_PNP_EBC, Q4 Q_PNP_EBC, Q5 Q_PNP_EBC, Q6 Q_PNP_EBC, Q7 Q_PNP_EBC, Q8 Q_PNP_EBC, Q9 Q_PNP_EBC, U31 74HC4051, U32 74HC4051, U33 74HC4051, U34 74HC4051

Commit message: started new project
Parts:
- added D1: LED, LED_SMD:LED_Everlight-SMD3528_3.5x2.8mm_67-21ST, F.Cu at (40.5, 127.0)
- added D10: LED, LED_SMD:LED_Everlight-SMD3528_3.5x2.8mm_67-21ST, F.Cu at (58.2, 70.0)
- added D11: LED, LED_SMD:LED_Everlight-SMD3528_3.5x2.8mm_67-21ST, F.Cu at (76.5, 49.5)
- added D12: LED, LED_SMD:LED_Everlight-SMD3528_3.5x2.8mm_67-21ST, F.Cu at (78.2, 70.0)
- added D13: LED, LED_SMD:LED_Everlight-SMD3528_3.5x2.8mm_67-21ST, F.Cu at (77.5, 89.0)
- added D14: LED, LED_SMD:LED_Everlight-SMD3528_3.5x2.8mm_67-21ST, F.Cu at (77.7, 107.5)
- added D15: LED, LED_SMD:LED_Everlight-SMD3528_3.5x2.8mm_67-21ST, F.Cu at (77.7, 126.0)
- added D16: LED, LED_SMD:LED_Everlight-SMD3528_3.5x2.8mm_67-21ST, F.Cu at (96.5, 49.5)
- added D17: LED, LED_SMD:LED_Everlight-SMD3528_3.5x2.8mm_67-21ST, F.Cu at (96.0, 70.0)
- added D18: LED, LED_SMD:LED_Everlight-SMD3528_3.5x2.8mm_67-21ST, F.Cu at (96.5, 88.5)
- added D19: LED, LED_SMD:LED_Everlight-SMD3528_3.5x2.8mm_67-21ST, F.Cu at (96.5, 107.0)
- added D2: LED, LED_SMD:LED_Everlight-SMD3528_3.5x2.8mm_67-21ST, F.Cu at (41.0, 107.0)
- added D20: LED, LED_SMD:LED_Everlight-SMD3528_3.5x2.8mm_67-21ST, F.Cu at (96.5, 126.0)
- added D21: LED, LED_SMD:LED_Everlight-SMD3528_3.5x2.8mm_67-21ST, F.Cu at (115.0, 49.5)
- added D22: LED, LED_SMD:LED_Everlight-SMD3528_3.5x2.8mm_67-21ST, F.Cu at (115.0, 69.5)
- added D23: LED, LED_SMD:LED_Everlight-SMD3528_3.5x2.8mm_67-21ST, F.Cu at (115.7, 88.5)
- added D24: LED, LED_SMD:LED_Everlight-SMD3528_3.5x2.8mm_67-21ST, F.Cu at (115.2, 106.5)
- added D25: LED, LED_SMD:LED_Everlight-SMD3528_3.5x2.8mm_67-21ST, F.Cu at (115.8, 126.5)
- added D26: LED, LED_SMD:LED_Everlight-SMD3528_3.5x2.8mm_67-21ST, F.Cu at (133.5, 49.0)
- added D27: LED, LED_SMD:LED_Everlight-SMD3528_3.5x2.8mm_67-21ST, F.Cu at (133.5, 68.0)
- added D28: LED, LED_SMD:LED_Everlight-SMD3528_3.5x2.8mm_67-21ST, F.Cu at (134.2, 87.0)
- added D29: LED, LED_SMD:LED_Everlight-SMD3528_3.5x2.8mm_67-21ST, F.Cu at (134.5, 106.5)
- added D3: LED, LED_SMD:LED_Everlight-SMD3528_3.5x2.8mm_67-21ST, F.Cu at (41.0, 88.5)
- added D30: LED, LED_SMD:LED_Everlight-SMD3528_3.5x2.8mm_67-21ST, F.Cu at (133.5, 125.0)
- added D4: LED, LED_SMD:LED_Everlight-SMD3528_3.5x2.8mm_67-21ST, F.Cu at (40.7, 68.0)
- added D5: LED, LED_SMD:LED_Everlight-SMD3528_3.5x2.8mm_67-21ST, F.Cu at (40.2, 49.5)
- added D6: LED, LED_SMD:LED_Everlight-SMD3528_3.5x2.8mm_67-21ST, F.Cu at (58.0, 49.5)
- added D7: LED, LED_SMD:LED_Everlight-SMD3528_3.5x2.8mm_67-21ST, F.Cu at (59.5, 127.0)
- added D8: LED, LED_SMD:LED_Everlight-SMD3528_3.5x2.8mm_67-21ST, F.Cu at (58.5, 107.0)
- added D9: LED, LED_SMD:LED_Everlight-SMD3528_3.5x2.8mm_67-21ST, F.Cu at (58.5, 89.0)
- added Q31: NMOS, Package_TO_SOT_SMD:SOT-23, F.Cu at (148.9, 97.5)
- added R1: R_Small, Resistor_SMD:R_1206_3216Metric_Pad1.30x1.75mm_HandSolder, F.Cu at (47.5, 130.0)
- added R10: R_Small, Resistor_SMD:R_1206_3216Metric_Pad1.30x1.75mm_HandSolder, F.Cu at (64.0, 70.0)
- added R11: R_Small, Resistor_SMD:R_1206_3216Metric_Pad1.30x1.75mm_HandSolder, F.Cu at (82.0, 49.5)
- added R12: R_Small, Resistor_SMD:R_1206_3216Metric_Pad1.30x1.75mm_HandSolder, F.Cu at (83.5, 70.5)
- added R13: R_Small, Resistor_SMD:R_1206_3216Metric_Pad1.30x1.75mm_HandSolder, F.Cu at (83.5, 89.5)
- added R14: R_Small, Resistor_SMD:R_1206_3216Metric_Pad1.30x1.75mm_HandSolder, F.Cu at (84.0, 107.5)
- added R15: R_Small, Resistor_SMD:R_1206_3216Metric_Pad1.30x1.75mm_HandSolder, F.Cu at (84.0, 126.0)
- added R16: R_Small, Resistor_SMD:R_1206_3216Metric_Pad1.30x1.75mm_HandSolder, F.Cu at (102.0, 49.5)
- added R17: R_Small, Resistor_SMD:R_1206_3216Metric_Pad1.30x1.75mm_HandSolder, F.Cu at (102.0, 70.0)
- added R18: R_Small, Resistor_SMD:R_1206_3216Metric_Pad1.30x1.75mm_HandSolder, F.Cu at (102.0, 88.5)
- added R19: R_Small, Resistor_SMD:R_1206_3216Metric_Pad1.30x1.75mm_HandSolder, F.Cu at (102.0, 107.0)
- added R2: R_Small, Resistor_SMD:R_1206_3216Metric_Pad1.30x1.75mm_HandSolder, F.Cu at (47.0, 107.0)
- added R20: R_Small, Resistor_SMD:R_1206_3216Metric_Pad1.30x1.75mm_HandSolder, F.Cu at (102.0, 126.0)
- added R21: R_Small, Resistor_SMD:R_1206_3216Metric_Pad1.30x1.75mm_HandSolder, F.Cu at (121.0, 49.5)
- added R22: R_Small, Resistor_SMD:R_1206_3216Metric_Pad1.30x1.75mm_HandSolder, F.Cu at (121.0, 69.5)
- added R23: R_Small, Resistor_SMD:R_1206_3216Metric_Pad1.30x1.75mm_HandSolder, F.Cu at (121.0, 88.5)
- added R24: R_Small, Resistor_SMD:R_1206_3216Metric_Pad1.30x1.75mm_HandSolder, F.Cu at (121.0, 106.5)
- added R25: R_Small, Resistor_SMD:R_1206_3216Metric_Pad1.30x1.75mm_HandSolder, F.Cu at (121.5, 126.5)
- added R26: R_Small, Resistor_SMD:R_1206_3216Metric_Pad1.30x1.75mm_HandSolder, F.Cu at (139.1, 49.0)
- added R27: R_Small, Resistor_SMD:R_1206_3216Metric_Pad1.30x1.75mm_HandSolder, F.Cu at (139.5, 68.0)
- added R28: R_Small, Resistor_SMD:R_1206_3216Metric_Pad1.30x1.75mm_HandSolder, F.Cu at (140.6, 87.5)
- added R29: R_Small, Resistor_SMD:R_1206_3216Metric_Pad1.30x1.75mm_HandSolder, F.Cu at (141.6, 106.5)
- added R3: R_Small, Resistor_SMD:R_1206_3216Metric_Pad1.30x1.75mm_HandSolder, F.Cu at (47.0, 88.5)
- added R30: R_Small, Resistor_SMD:R_1206_3216Metric_Pad1.30x1.75mm_HandSolder, F.Cu at (142.1, 125.5)
- added R4: R_Small, Resistor_SMD:R_1206_3216Metric_Pad1.30x1.75mm_HandSolder, F.Cu at (47.0, 67.5)
- added R5: R_Small, Resistor_SMD:R_1206_3216Metric_Pad1.30x1.75mm_HandSolder, F.Cu at (47.0, 49.5)
- added R6: R_Small, Resistor_SMD:R_1206_3216Metric_Pad1.30x1.75mm_HandSolder, F.Cu at (64.5, 49.5)
- added R7: R_Small, Resistor_SMD:R_1206_3216Metric_Pad1.30x1.75mm_HandSolder, F.Cu at (65.0, 128.0)
- added R8: R_Small, Resistor_SMD:R_1206_3216Metric_Pad1.30x1.75mm_HandSolder, F.Cu at (64.5, 107.0)
- added R9: R_Small, Resistor_SMD:R_1206_3216Metric_Pad1.30x1.75mm_HandSolder, F.Cu at (64.0, 89.0)
- U31, U32, U33, U34: footprint Package_DIP:DIP-16_W7.62mm -> Package_SO:SOIC-16_3.9x9.9mm_P1.27mm; moved to B.Cu
- moved U31 145.6 mm to (161.6, 135.5), turned to 90 degrees
- moved U32 129.5 mm to (161.6, 123.6), turned to 90 degrees
- moved A1 116.1 mm to (161.5, 67.5)
- moved U33 114.1 mm to (161.6, 112.5), turned to 90 degrees
- moved U34 98.3 mm to (161.8, 100.8), turned to 90 degrees
- moved Q26 85.6 mm to (58.0, 133.2)
- moved Q27 74.2 mm to (77.1, 133.2)
- moved Q25 72.5 mm to (39.0, 133.2)
- moved Q30 69.2 mm to (134.2, 133.2)
- moved Q6 67.9 mm to (134.2, 57.0)
- moved Q28 66.9 mm to (96.2, 133.2)
- moved Q29 65.1 mm to (115.2, 133.2)
- moved Q24 64.0 mm to (134.2, 114.2)
- moved Q12 63.2 mm to (134.2, 76.0)
- moved Q16 63.0 mm to (58.0, 114.2)
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Connections:
- A1 pad 20: unconnected-(A1-GPIO15-Pad20) -> Net-(A1-GPIO15)
- A1 pad 39: unconnected-(A1-VSYS-Pad39) -> Net-(A1-VSYS)
